File: PCB design/Template_PiggyBack.sch (EAGLE design)
At the start: 27 parts, among them CN1 USB power supply, IC1 MCP6002, IC2 Hall-Sensor-DRV5053VA, IC4 REG1117

Commit message: circuit sketch done
Parts:
- added C10: 22µ, rcl:C-EUC0805
- added IC3: MCP6002, linear:OPA2333D
- added R2, R5: 3.3k, rcl:R-EU_R0805
- added R3, R6, R7: 100, rcl:R-EU_R0805
- added R4, R8: 3k, rcl:R-EU_R0805
- added TP_GND: PTR1PAD1-17, testpad:PTR1PAD1-17
- C1: value 100u -> 22n
- C2: value 10u -> 4.7n
- C3: value 1u -> 22µ
- C8: value 100n -> 10µ
- C9: value 10n -> 4.7n
- R1: value (none) -> 100k
Connections:
- new net N$10: C1.1
- new net N$2: C2.1, C3.2, IC1B.-IN, R2.1, R3.1, R3.2
- new net N$3: C10.2, R7.1
- new net N$4: C1.2, IC1B.+IN, R1.2
- new net N$5: C2.2, IC1B.OUT, IC3B.+IN, R2.2
- new net N$6: C8.1, R4.1, R8.2
- new net N$7: C9.2, IC3B.OUT, R5.2, R6.1
- new net N$8: C9.1, IC3B.-IN, R5.1, R7.2
- new net N$9: R6.2
- new net VCC: R4.2
- new net V_GND: R1.1
- net GND: now also C10.1, C3.1, C8.2, R8.1, TP_GND.TP
Other:
- moved on the sheet: C1, C2, C3, C8, C9, IC1B, R1
